File: KiCAD/CIB - Flapjack Octopus.kicad_pcb (KiCad board)
At the start: 2 copper layers, 83 x 133 mm, 117 parts, among them J1 CIO0, J10 CIO2, J11 EIO4, J12 FIO2, J13 MIO0, J14 CIO3, J15 EIO5, J16 FIO3, J17 MIO1, J18 EIO0, J19 EIO6, J2 EIO2, J20 FIO4, J21 MIO2, J22 DC37, J23 EIO7, J24 FIO5, J25 EIO1, J26 CIO, J27 MIO, J28 EIO, J29 FIO, J3 FIO0, J30 AIN0, J31 AIN1, J32 AIN2, J33 AIN3, J34 AIN6, J35 AIN9, J36 AIN12, J37 AIN4, J38 AIN7, J39 AIN10, J4 FIO6, J40 AIN13, J41 AIN5, J42 AIN8, J43 AIN11, J44 5V, J45 GND, J46 AIN, J47 AIN, J48 External Supply, J49 Relays, J5 DA15, J50 MISC, J6 CIO1, J7 EIO3, J8 FIO1, J9 FIO7, U1 74LS04, U2 74LS04, U3 74LS04, U4 74LS04, U5 ULN2803A

Commit message: .
Parts:
- moved R37 0.73 mm to (97.2, 29.8)
- moved JP1 0.17 mm to (97.2, 27.2)
Routing:
- net GND: track 100.3 -> 99.1 mm, vias 6 -> 5
- net Net-(J49-Pin_6): track 10.2 -> 9.32 mm
- net +5V: track 50.1 -> 49.3 mm
- net /EIO1: track 75.8 -> 75.1 mm
- net Net-(R19-Pad1): track 7.46 -> 6.85 mm
- net +5V5_ISO_1: track 89.3 -> 88.8 mm

Commit message: .
Connections:
- net +5V5_ISO_1 renamed +5V_ISO

Commit message: .
Parts:
- removed D1: EIO2, LED_SMD:LED_0805_2012Metric_Pad1.15x1.40mm_HandSolder
- removed D2: EIO3, LED_SMD:LED_0805_2012Metric_Pad1.15x1.40mm_HandSolder
- removed D3: EIO4, LED_SMD:LED_0805_2012Metric_Pad1.15x1.40mm_HandSolder
- removed D4: EIO5, LED_SMD:LED_0805_2012Metric_Pad1.15x1.40mm_HandSolder
- removed D5: EIO7, LED_SMD:LED_0805_2012Metric_Pad1.15x1.40mm_HandSolder
- removed D6: EIO6, LED_SMD:LED_0805_2012Metric_Pad1.15x1.40mm_HandSolder
- removed J1: CIO0, Connector_PinSocket_2.54mm:PinSocket_1x03_P2.54mm_Vertical
- removed J10: CIO2, Connector_PinSocket_2.54mm:PinSocket_1x03_P2.54mm_Vertical
- removed J11: EIO4, Connector_PinSocket_2.54mm:PinSocket_1x03_P2.54mm_Vertical
- removed J12: FIO2, Connector_PinSocket_2.54mm:PinSocket_1x03_P2.54mm_Vertical
- removed J13: MIO0, Connector_PinSocket_2.54mm:PinSocket_1x03_P2.54mm_Vertical
- removed J14: CIO3, Connector_PinSocket_2.54mm:PinSocket_1x03_P2.54mm_Vertical
- removed J15: EIO5, Connector_PinSocket_2.54mm:PinSocket_1x03_P2.54mm_Vertical
- removed J16: FIO3, Connector_PinSocket_2.54mm:PinSocket_1x03_P2.54mm_Vertical
- removed J17: MIO1, Connector_PinSocket_2.54mm:PinSocket_1x03_P2.54mm_Vertical
- removed J18: EIO0, Connector_PinSocket_2.54mm:PinSocket_1x03_P2.54mm_Vertical
- removed J19: EIO6, Connector_PinSocket_2.54mm:PinSocket_1x03_P2.54mm_Vertical
- removed J2: EIO2, Connector_PinSocket_2.54mm:PinSocket_1x03_P2.54mm_Vertical
- removed J20: FIO4, Connector_PinSocket_2.54mm:PinSocket_1x03_P2.54mm_Vertical
- removed J21: MIO2, Connector_PinSocket_2.54mm:PinSocket_1x03_P2.54mm_Vertical
- removed J23: EIO7, Connector_PinSocket_2.54mm:PinSocket_1x03_P2.54mm_Vertical
- removed J24: FIO5, Connector_PinSocket_2.54mm:PinSocket_1x03_P2.54mm_Vertical
- removed J25: EIO1, Connector_PinSocket_2.54mm:PinSocket_1x03_P2.54mm_Vertical
- removed J3: FIO0, Connector_PinSocket_2.54mm:PinSocket_1x03_P2.54mm_Vertical
- removed J36: AIN12, Connector_PinSocket_2.54mm:PinSocket_1x03_P2.54mm_Vertical
- removed J37: AIN4, Connector_PinSocket_2.54mm:PinSocket_1x03_P2.54mm_Vertical
- removed J38: AIN7, Connector_PinSocket_2.54mm:PinSocket_1x03_P2.54mm_Vertical
- removed J39: AIN10, Connector_PinSocket_2.54mm:PinSocket_1x03_P2.54mm_Vertical
- removed J4: FIO6, Connector_PinSocket_2.54mm:PinSocket_1x03_P2.54mm_Vertical
- removed J40: AIN13, Connector_PinSocket_2.54mm:PinSocket_1x03_P2.54mm_Vertical
- removed J41: AIN5, Connector_PinSocket_2.54mm:PinSocket_1x03_P2.54mm_Vertical
- removed J42: AIN8, Connector_PinSocket_2.54mm:PinSocket_1x03_P2.54mm_Vertical
- removed J43: AIN11, Connector_PinSocket_2.54mm:PinSocket_1x03_P2.54mm_Vertical
- removed J6: CIO1, Connector_PinSocket_2.54mm:PinSocket_1x03_P2.54mm_Vertical
- removed J7: EIO3, Connector_PinSocket_2.54mm:PinSocket_1x03_P2.54mm_Vertical
- removed J8: FIO1, Connector_PinSocket_2.54mm:PinSocket_1x03_P2.54mm_Vertical
- removed J9: FIO7, Connector_PinSocket_2.54mm:PinSocket_1x03_P2.54mm_Vertical
- removed R1, R2, R3, R31, R32, R35, R36, R4, R5, R6: 1k, Resistor_SMD:R_0805_2012Metric_Pad1.20x1.40mm_HandSolder
- removed R33, R34: 2k2, Resistor_SMD:R_0805_2012Metric_Pad1.20x1.40mm_HandSolder
- removed U1: 74LS04, Package_SO:SSOP-14_5.3x6.2mm_P0.65mm
- added D25: GN, LED_SMD:LED_0805_2012Metric_Pad1.15x1.40mm_HandSolder, F.Cu at (190.6, 102.1)
- added D26: GN, LED_SMD:LED_0805_2012Metric_Pad1.15x1.40mm_HandSolder, F.Cu at (190.6, 105.2)
- added D27: GN, LED_SMD:LED_0805_2012Metric_Pad1.15x1.40mm_HandSolder, F.Cu at (190.6, 108.2)
- added D28: GN, LED_SMD:LED_0805_2012Metric_Pad1.15x1.40mm_HandSolder, F.Cu at (190.6, 111.3)
- added D29: GN, LED_SMD:LED_0805_2012Metric_Pad1.15x1.40mm_HandSolder, F.Cu at (190.6, 114.3)
- added D30: GN, LED_SMD:LED_0805_2012Metric_Pad1.15x1.40mm_HandSolder, F.Cu at (190.6, 117.3)
- added J51: Conn_01x06_Pin, Connector_PinHeader_2.54mm:PinHeader_1x06_P2.54mm_Vertical, F.Cu at (149.2, 97.2)
- added J52: Conn_01x06_Pin, Connector_PinHeader_2.54mm:PinHeader_1x06_P2.54mm_Vertical, F.Cu at (149.2, 117.5)
- added J53: Conn_01x06_Pin, Connector_PinHeader_2.54mm:PinHeader_1x06_P2.54mm_Vertical, F.Cu at (151.8, 97.2)
- added J54: Conn_01x06_Pin, Connector_PinHeader_2.54mm:PinHeader_1x06_P2.54mm_Vertical, F.Cu at (151.8, 117.5)
- added J55: Conn_01x06_Pin, Connector_PinHeader_2.54mm:PinHeader_1x06_P2.54mm_Vertical, F.Cu at (154.3, 97.2)
- added J56: Conn_01x06_Pin, Connector_PinHeader_2.54mm:PinHeader_1x06_P2.54mm_Vertical, F.Cu at (154.3, 117.5)
- added J57: Conn_01x04_Pin, Connector_PinHeader_2.54mm:PinHeader_1x04_P2.54mm_Vertical, F.Cu at (149.2, 18.4)
- added J58: Conn_01x08_Pin, Connector_PinHeader_2.54mm:PinHeader_1x08_P2.54mm_Vertical, F.Cu at (149.2, 33.7)
- added J59: Conn_01x08_Pin, Connector_PinHeader_2.54mm:PinHeader_1x08_P2.54mm_Vertical, F.Cu at (149.2, 59.1)
- added J60: Conn_01x04_Pin, Connector_PinHeader_2.54mm:PinHeader_1x04_P2.54mm_Vertical, F.Cu at (151.8, 18.3)
- added J61: Conn_01x04_Pin, Connector_PinHeader_2.54mm:PinHeader_1x04_P2.54mm_Vertical, F.Cu at (154.3, 18.4)
- added J62: Conn_01x08_Pin, Connector_PinHeader_2.54mm:PinHeader_1x08_P2.54mm_Vertical, F.Cu at (151.8, 33.7)
- added J63: Conn_01x08_Pin, Connector_PinHeader_2.54mm:PinHeader_1x08_P2.54mm_Vertical, F.Cu at (154.3, 33.7)
- added J64: Conn_01x08_Pin, Connector_PinHeader_2.54mm:PinHeader_1x08_P2.54mm_Vertical, F.Cu at (151.8, 59.1)
- added J65: Conn_01x08_Pin, Connector_PinHeader_2.54mm:PinHeader_1x08_P2.54mm_Vertical, F.Cu at (154.3, 59.1)
- added JP10: A1, Jumper:SolderJumper-2_P1.3mm_Bridged_RoundedPad1.0x1.5mm, F.Cu at (137.8, 128.3)
- added JP11: A1 AG, Jumper:SolderJumper-2_P1.3mm_Open_RoundedPad1.0x1.5mm, F.Cu at (118.1, 128.3)
- added JP12: A1, Jumper:SolderJumper-2_P1.3mm_Bridged_RoundedPad1.0x1.5mm, F.Cu at (137.8, 131.4)
- added JP13: A1 AG, Jumper:SolderJumper-2_P1.3mm_Open_RoundedPad1.0x1.5mm, F.Cu at (118.1, 131.4)
- added JP14: A1, Jumper:SolderJumper-2_P1.3mm_Bridged_RoundedPad1.0x1.5mm, F.Cu at (137.8, 134.6)
- added JP15: A1 AG, Jumper:SolderJumper-2_P1.3mm_Open_RoundedPad1.0x1.5mm, F.Cu at (118.1, 134.6)
- added JP16: A1, Jumper:SolderJumper-2_P1.3mm_Bridged_RoundedPad1.0x1.5mm, F.Cu at (137.8, 137.8)
- added JP17: A1 AG, Jumper:SolderJumper-2_P1.3mm_Open_RoundedPad1.0x1.5mm, F.Cu at (118.1, 137.8)
- added JP6: A1, Jumper:SolderJumper-2_P1.3mm_Bridged_RoundedPad1.0x1.5mm, F.Cu at (137.8, 121.9)
- added JP7: A1 AG, Jumper:SolderJumper-2_P1.3mm_Open_RoundedPad1.0x1.5mm, F.Cu at (118.1, 121.9)
- added JP8: A1, Jumper:SolderJumper-2_P1.3mm_Bridged_RoundedPad1.0x1.5mm, F.Cu at (137.8, 125.1)
- added JP9: A1 AG, Jumper:SolderJumper-2_P1.3mm_Open_RoundedPad1.0x1.5mm, F.Cu at (118.1, 125.1)
- added R1a10: THT, Resistor_THT:R_Axial_DIN0207_L6.3mm_D2.5mm_P10.16mm_Horizontal, F.Cu at (144.8, 131.4)
- added R1a11: SMD, Resistor_SMD:R_0805_2012Metric_Pad1.20x1.40mm_HandSolder, F.Cu at (141.6, 134.6)
- added R1a12: THT, Resistor_THT:R_Axial_DIN0207_L6.3mm_D2.5mm_P10.16mm_Horizontal, F.Cu at (144.8, 134.6)
- added R1a13: SMD, Resistor_SMD:R_0805_2012Metric_Pad1.20x1.40mm_HandSolder, F.Cu at (141.6, 137.8)
- added R1a14: THT, Resistor_THT:R_Axial_DIN0207_L6.3mm_D2.5mm_P10.16mm_Horizontal, F.Cu at (144.8, 137.8)
- added R1a3: SMD, Resistor_SMD:R_0805_2012Metric_Pad1.20x1.40mm_HandSolder, F.Cu at (141.6, 121.9)
- added R1a4: THT, Resistor_THT:R_Axial_DIN0207_L6.3mm_D2.5mm_P10.16mm_Horizontal, F.Cu at (144.8, 121.9)
- added R1a5: SMD, Resistor_SMD:R_0805_2012Metric_Pad1.20x1.40mm_HandSolder, F.Cu at (141.6, 125.1)
- added R1a6: THT, Resistor_THT:R_Axial_DIN0207_L6.3mm_D2.5mm_P10.16mm_Horizontal, F.Cu at (144.8, 125.1)
- added R1a7: SMD, Resistor_SMD:R_0805_2012Metric_Pad1.20x1.40mm_HandSolder, F.Cu at (141.6, 128.3)
- added R1a8: THT, Resistor_THT:R_Axial_DIN0207_L6.3mm_D2.5mm_P10.16mm_Horizontal, F.Cu at (144.8, 128.3)
- added R1a9: SMD, Resistor_SMD:R_0805_2012Metric_Pad1.20x1.40mm_HandSolder, F.Cu at (141.6, 131.4)
- added R1b10: THT, Resistor_THT:R_Axial_DIN0207_L6.3mm_D2.5mm_P10.16mm_Horizontal, F.Cu at (132.1, 131.4)
- added R1b11: SMD, Resistor_SMD:R_0805_2012Metric_Pad1.20x1.40mm_HandSolder, F.Cu at (127.0, 134.6)
- added R1b12: THT, Resistor_THT:R_Axial_DIN0207_L6.3mm_D2.5mm_P10.16mm_Horizontal, F.Cu at (132.1, 134.6)
- added R1b13: SMD, Resistor_SMD:R_0805_2012Metric_Pad1.20x1.40mm_HandSolder, F.Cu at (127.0, 137.8)
- added R1b14: THT, Resistor_THT:R_Axial_DIN0207_L6.3mm_D2.5mm_P10.16mm_Horizontal, F.Cu at (132.1, 137.8)
- added R1b3: SMD, Resistor_SMD:R_0805_2012Metric_Pad1.20x1.40mm_HandSolder, F.Cu at (127.0, 121.9)
- added R1b4: THT, Resistor_THT:R_Axial_DIN0207_L6.3mm_D2.5mm_P10.16mm_Horizontal, F.Cu at (132.1, 121.9)
- added R1b5: SMD, Resistor_SMD:R_0805_2012Metric_Pad1.20x1.40mm_HandSolder, F.Cu at (127.0, 125.1)
- added R1b6: THT, Resistor_THT:R_Axial_DIN0207_L6.3mm_D2.5mm_P10.16mm_Horizontal, F.Cu at (132.1, 125.1)
- added R1b7: SMD, Resistor_SMD:R_0805_2012Metric_Pad1.20x1.40mm_HandSolder, F.Cu at (127.0, 128.3)
- added R1b8: THT, Resistor_THT:R_Axial_DIN0207_L6.3mm_D2.5mm_P10.16mm_Horizontal, F.Cu at (132.1, 128.3)
- added R1b9: SMD, Resistor_SMD:R_0805_2012Metric_Pad1.20x1.40mm_HandSolder, F.Cu at (127.0, 131.4)
- added U6: 74LS04, Package_SO:SSOP-14_5.3x6.2mm_P0.65mm, F.Cu at (174.6, 81.3)
- D10: value CIO1 -> GN
- D11: value FIO1 -> GN
- D12: value FIO7 -> GN
- D13: value CIO2 -> GN
- D14: value FIO2 -> GN
- D15: value MIO0 -> GN
- D16: value CIO3 -> GN
- D17: value FIO3 -> GN
- D18: value MIO1 -> GN
- D19: value EIO0 -> GN
- D20: value FIO4 -> GN
- D21: value MIO2 -> GN
- D22: value EIO1 -> GN
- D23: value FIO5 -> GN
- D24: value Power -> GN
- D7: value CIO0 -> GN
- D8: value FIO0 -> GN
- D9: value FIO6 -> GN
- J30: value AIN0 -> Conn_01x02_Pin; footprint Connector_PinSocket_2.54mm:PinSocket_1x03_P2.54mm_Vertical -> Connector_PinSocket_2.54mm:PinSocket_1x02_P2.54mm_Vertical
- J31: value AIN1 -> Conn_01x02_Pin; footprint Connector_PinSocket_2.54mm:PinSocket_1x03_P2.54mm_Vertical -> Connector_PinSocket_2.54mm:PinSocket_1x02_P2.54mm_Vertical
- J32: value AIN2 -> Conn_01x02_Pin; footprint Connector_PinSocket_2.54mm:PinSocket_1x03_P2.54mm_Vertical -> Connector_PinSocket_2.54mm:PinSocket_1x02_P2.54mm_Vertical
- J33: value AIN3 -> CIO0
- J34: value AIN6 -> CIO0
- J35: value AIN9 -> CIO0
- R25, R26, R29, R30: value 2k2 -> 1k
- R37: value 1k -> 0
- moved D11 73.6 mm to (212.1, 49.5)
- moved D12 73.6 mm to (212.1, 64.8)
- moved D14 73.6 mm to (212.1, 52.1)
- moved D17 73.6 mm to (212.1, 54.6)
- moved D20 73.6 mm to (212.1, 57.1)
- moved D23 73.6 mm to (212.1, 59.7)
- moved D8 73.6 mm to (212.1, 47.0)
- moved D9 73.6 mm to (212.1, 62.2)
- moved R11 73.6 mm to (207.0, 49.5)
- moved R12 73.6 mm to (207.0, 64.8)
- moved R14 73.6 mm to (207.0, 52.1)
- moved R17 73.6 mm to (207.0, 54.6)
- moved R20 73.6 mm to (207.0, 57.1)
- moved R23 73.6 mm to (207.0, 59.7)
- moved R8 73.6 mm to (207.0, 47.0)
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Connections:
- J30 pad 1: /AIN0 -> /AIN12_PD
- J30 pad 2: +5V -> /AIN13_PD
- J31 pad 1: /AIN1 -> +5V
- J32 pad 1: /AIN2 -> GND
- J32 pad 2: +5V -> GND
- J33 pad 1: /AIN3 -> /MIO0
- J33 pad 2: +5V -> /MIO1
- J33 pad 3: GND -> /MIO2
- J34 pad 1: /AIN6 -> +5V
- J34 pad 3: GND -> +5V
- J35 pad 1: Net-(J35-Pin_1) -> GND
- J35 pad 2: /AIN9 -> GND
- J47 pad 1: /AIN13 -> /AIN13_PD
- J47 pad 2: /AIN12 -> /AIN12_PD
- J47 pad 3: /AIN11 -> /AIN11_PD
- J47 pad 4: /AIN10 -> /AIN10_PD
- J47 pad 5: /AIN9 -> /AIN9_PD
- J47 pad 6: /AIN8 -> /AIN8_PD
- R25 pad 1: /AIN9 -> Net-(R25-Pad1)
- R25 pad 2: Net-(J35-Pin_1) -> Net-(D25-K)
- R26 pad 1: /AIN12 -> Net-(R26-Pad1)
- R27 pad 1: /AIN9 -> Net-(R27-Pad1)
- R27 pad 2: GND -> Net-(D27-K)
- R28 pad 1: /AIN12 -> Net-(R28-Pad1)
- R28 pad 2: GND -> Net-(D28-K)
- R29 pad 1: /AIN10 -> Net-(R29-Pad1)
- R30 pad 1: /AIN13 -> Net-(R30-Pad1)
- U2 pad 14: +5V -> (no net)
- U2 pad 7: GND -> (no net)
- U3 pad 1: /FIO1 -> /EIO3
- U3 pad 10: Net-(R20-Pad1) -> Net-(R23-Pad1)
- U3 pad 11: /FIO4 -> /EIO7
- U3 pad 12: Net-(R17-Pad1) -> Net-(R20-Pad1)
- U3 pad 13: /FIO3 -> /EIO6
- U3 pad 14: +5V -> (no net)
- U3 pad 3: /FIO0 -> /EIO2
- U3 pad 5: /FIO2 -> /EIO4
- U3 pad 7: GND -> (no net)
- U3 pad 8: Net-(R23-Pad1) -> Net-(R17-Pad1)
- U3 pad 9: /FIO5 -> /EIO5
- U4 pad 1: /FIO7 -> /FIO1
- U4 pad 10: Net-(R21-Pad1) -> Net-(R24-Pad1)
- U4 pad 11: /MIO2 -> /FIO5
- U4 pad 12: Net-(R18-Pad1) -> Net-(R21-Pad1)
- U4 pad 13: /MIO1 -> /FIO4
- U4 pad 3: /FIO6 -> /FIO0
- U4 pad 5: /MIO0 -> /FIO2
- U4 pad 8: Net-(R24-Pad1) -> Net-(R18-Pad1)
- U4 pad 9: +5V -> /FIO3
Routing:
- net +5V: track 49.3 -> 256.6 mm, vias 29 -> 2
- net /AIN11: track 109.5 -> 13.8 mm, vias 1 -> 0
- net /AIN10: track 108.5 -> 13.8 mm, vias 1 -> 0
- net GND: track 99.1 -> 8.10 mm, vias 5 -> 1
- net /CIO0: track 100.5 -> 11.7 mm
- net /AIN9: track 101.0 -> 13.8 mm, vias 1 -> 0
- net /CIO2: track 98.5 -> 11.7 mm
- net /CIO1: track 93.3 -> 11.8 mm
- net Net-(R24-Pad1): track 73.2 -> 0.00 mm
- net /MIO0: track 83.4 -> 11.7 mm, vias 1 -> 0
- net /MIO2: track 82.5 -> 11.7 mm, vias 1 -> 0
- net /EIO7: track 80.1 -> 11.7 mm, vias 1 -> 0
- net /EIO5: track 78.0 -> 11.7 mm, vias 1 -> 0
- net /MIO1: track 77.4 -> 11.7 mm, vias 1 -> 0
- net /EIO2: track 77.1 -> 11.8 mm, vias 1 -> 0
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- added copper zone on B.Cu, net GND
- removed copper zone on B.Cu, net +5V
