File: KiCAD/CIB - Flapjack Octopus.kicad_sch (KiCad schematic)
At the start: 117 parts, among them J1 CIO0, J10 CIO2, J11 EIO4, J12 FIO2, J13 MIO0, J14 CIO3, J15 EIO5, J16 FIO3, J17 MIO1, J18 EIO0, J19 EIO6, J2 EIO2, J20 FIO4, J21 MIO2, J22 DC37, J23 EIO7, J24 FIO5, J25 EIO1, J26 CIO, J27 MIO, J28 EIO, J29 FIO, J3 FIO0, J30 AIN0, J31 AIN1, J32 AIN2, J33 AIN3, J34 AIN6, J35 AIN9, J36 AIN12, J37 AIN4, J38 AIN7, J39 AIN10, J4 FIO6, J40 AIN13, J41 AIN5, J42 AIN8, J43 AIN11, J44 5V, J45 GND, J46 AIN, J47 AIN, J48 External Supply, J49 Relays, J5 DA15, J50 MISC, J6 CIO1, J7 EIO3, J8 FIO1, J9 FIO7, U1 74LS04, U2 74LS04, U3 74LS04, U4 74LS04, U5 ULN2803A

Commit message: .
Connections:
- net +5V5_ISO_1 renamed +5V_ISO

Commit message: .
Parts:
- removed D1: EIO2, LED_SMD:LED_0805_2012Metric_Pad1.15x1.40mm_HandSolder, symbol Device:LED_Small_Filled
- removed D10: CIO1, LED_SMD:LED_0805_2012Metric_Pad1.15x1.40mm_HandSolder, symbol Device:LED_Small_Filled
- removed D11: FIO1, LED_SMD:LED_0805_2012Metric_Pad1.15x1.40mm_HandSolder, symbol Device:LED_Small_Filled
- removed D12: FIO7, LED_SMD:LED_0805_2012Metric_Pad1.15x1.40mm_HandSolder, symbol Device:LED_Small_Filled
- removed D13: CIO2, LED_SMD:LED_0805_2012Metric_Pad1.15x1.40mm_HandSolder, symbol Device:LED_Small_Filled
- removed D14: FIO2, LED_SMD:LED_0805_2012Metric_Pad1.15x1.40mm_HandSolder, symbol Device:LED_Small_Filled
- removed D15: MIO0, LED_SMD:LED_0805_2012Metric_Pad1.15x1.40mm_HandSolder, symbol Device:LED_Small_Filled
- removed D16: CIO3, LED_SMD:LED_0805_2012Metric_Pad1.15x1.40mm_HandSolder, symbol Device:LED_Small_Filled
- removed D17: FIO3, LED_SMD:LED_0805_2012Metric_Pad1.15x1.40mm_HandSolder, symbol Device:LED_Small_Filled
- removed D18: MIO1, LED_SMD:LED_0805_2012Metric_Pad1.15x1.40mm_HandSolder, symbol Device:LED_Small_Filled
- removed D19: EIO0, LED_SMD:LED_0805_2012Metric_Pad1.15x1.40mm_HandSolder, symbol Device:LED_Small_Filled
- removed D2: EIO3, LED_SMD:LED_0805_2012Metric_Pad1.15x1.40mm_HandSolder, symbol Device:LED_Small_Filled
- removed D20: FIO4, LED_SMD:LED_0805_2012Metric_Pad1.15x1.40mm_HandSolder, symbol Device:LED_Small_Filled
- removed D21: MIO2, LED_SMD:LED_0805_2012Metric_Pad1.15x1.40mm_HandSolder, symbol Device:LED_Small_Filled
- removed D22: EIO1, LED_SMD:LED_0805_2012Metric_Pad1.15x1.40mm_HandSolder, symbol Device:LED_Small_Filled
- removed D23: FIO5, LED_SMD:LED_0805_2012Metric_Pad1.15x1.40mm_HandSolder, symbol Device:LED_Small_Filled
- removed D24: Power, LED_SMD:LED_0805_2012Metric_Pad1.15x1.40mm_HandSolder, symbol Device:LED_Small_Filled
- removed D3: EIO4, LED_SMD:LED_0805_2012Metric_Pad1.15x1.40mm_HandSolder, symbol Device:LED_Small_Filled
- removed D4: EIO5, LED_SMD:LED_0805_2012Metric_Pad1.15x1.40mm_HandSolder, symbol Device:LED_Small_Filled
- removed D5: EIO7, LED_SMD:LED_0805_2012Metric_Pad1.15x1.40mm_HandSolder, symbol Device:LED_Small_Filled
- removed D6: EIO6, LED_SMD:LED_0805_2012Metric_Pad1.15x1.40mm_HandSolder, symbol Device:LED_Small_Filled
- removed D7: CIO0, LED_SMD:LED_0805_2012Metric_Pad1.15x1.40mm_HandSolder, symbol Device:LED_Small_Filled
- removed D8: FIO0, LED_SMD:LED_0805_2012Metric_Pad1.15x1.40mm_HandSolder, symbol Device:LED_Small_Filled
- removed D9: FIO6, LED_SMD:LED_0805_2012Metric_Pad1.15x1.40mm_HandSolder, symbol Device:LED_Small_Filled
- removed J1: CIO0, Connector_PinSocket_2.54mm:PinSocket_1x03_P2.54mm_Vertical, symbol Connector:Conn_01x03_Pin
- removed J10: CIO2, Connector_PinSocket_2.54mm:PinSocket_1x03_P2.54mm_Vertical, symbol Connector:Conn_01x03_Pin
- removed J11: EIO4, Connector_PinSocket_2.54mm:PinSocket_1x03_P2.54mm_Vertical, symbol Connector:Conn_01x03_Pin
- removed J12: FIO2, Connector_PinSocket_2.54mm:PinSocket_1x03_P2.54mm_Vertical, symbol Connector:Conn_01x03_Pin
- removed J13: MIO0, Connector_PinSocket_2.54mm:PinSocket_1x03_P2.54mm_Vertical, symbol Connector:Conn_01x03_Pin
- removed J14: CIO3, Connector_PinSocket_2.54mm:PinSocket_1x03_P2.54mm_Vertical, symbol Connector:Conn_01x03_Pin
- removed J15: EIO5, Connector_PinSocket_2.54mm:PinSocket_1x03_P2.54mm_Vertical, symbol Connector:Conn_01x03_Pin
- removed J16: FIO3, Connector_PinSocket_2.54mm:PinSocket_1x03_P2.54mm_Vertical, symbol Connector:Conn_01x03_Pin
- removed J17: MIO1, Connector_PinSocket_2.54mm:PinSocket_1x03_P2.54mm_Vertical, symbol Connector:Conn_01x03_Pin
- removed J18: EIO0, Connector_PinSocket_2.54mm:PinSocket_1x03_P2.54mm_Vertical, symbol Connector:Conn_01x03_Pin
- removed J19: EIO6, Connector_PinSocket_2.54mm:PinSocket_1x03_P2.54mm_Vertical, symbol Connector:Conn_01x03_Pin
- removed J2: EIO2, Connector_PinSocket_2.54mm:PinSocket_1x03_P2.54mm_Vertical, symbol Connector:Conn_01x03_Pin
- removed J20: FIO4, Connector_PinSocket_2.54mm:PinSocket_1x03_P2.54mm_Vertical, symbol Connector:Conn_01x03_Pin
- removed J21: MIO2, Connector_PinSocket_2.54mm:PinSocket_1x03_P2.54mm_Vertical, symbol Connector:Conn_01x03_Pin
- removed J23: EIO7, Connector_PinSocket_2.54mm:PinSocket_1x03_P2.54mm_Vertical, symbol Connector:Conn_01x03_Pin
- removed J24: FIO5, Connector_PinSocket_2.54mm:PinSocket_1x03_P2.54mm_Vertical, symbol Connector:Conn_01x03_Pin
- removed J25: EIO1, Connector_PinSocket_2.54mm:PinSocket_1x03_P2.54mm_Vertical, symbol Connector:Conn_01x03_Pin
- removed J3: FIO0, Connector_PinSocket_2.54mm:PinSocket_1x03_P2.54mm_Vertical, symbol Connector:Conn_01x03_Pin
- removed J30: AIN0, Connector_PinSocket_2.54mm:PinSocket_1x03_P2.54mm_Vertical, symbol Connector:Conn_01x03_Pin
- removed J31: AIN1, Connector_PinSocket_2.54mm:PinSocket_1x03_P2.54mm_Vertical, symbol Connector:Conn_01x03_Pin
- removed J32: AIN2, Connector_PinSocket_2.54mm:PinSocket_1x03_P2.54mm_Vertical, symbol Connector:Conn_01x03_Pin
- removed J36: AIN12, Connector_PinSocket_2.54mm:PinSocket_1x03_P2.54mm_Vertical, symbol Connector:Conn_01x03_Pin
- removed J37: AIN4, Connector_PinSocket_2.54mm:PinSocket_1x03_P2.54mm_Vertical, symbol Connector:Conn_01x03_Pin
- removed J38: AIN7, Connector_PinSocket_2.54mm:PinSocket_1x03_P2.54mm_Vertical, symbol Connector:Conn_01x03_Pin
- removed J39: AIN10, Connector_PinSocket_2.54mm:PinSocket_1x03_P2.54mm_Vertical, symbol Connector:Conn_01x03_Pin
- removed J4: FIO6, Connector_PinSocket_2.54mm:PinSocket_1x03_P2.54mm_Vertical, symbol Connector:Conn_01x03_Pin
- removed J40: AIN13, Connector_PinSocket_2.54mm:PinSocket_1x03_P2.54mm_Vertical, symbol Connector:Conn_01x03_Pin
- removed J41: AIN5, Connector_PinSocket_2.54mm:PinSocket_1x03_P2.54mm_Vertical, symbol Connector:Conn_01x03_Pin
- removed J42: AIN8, Connector_PinSocket_2.54mm:PinSocket_1x03_P2.54mm_Vertical, symbol Connector:Conn_01x03_Pin
- removed J43: AIN11, Connector_PinSocket_2.54mm:PinSocket_1x03_P2.54mm_Vertical, symbol Connector:Conn_01x03_Pin
- removed J6: CIO1, Connector_PinSocket_2.54mm:PinSocket_1x03_P2.54mm_Vertical, symbol Connector:Conn_01x03_Pin
- removed J7: EIO3, Connector_PinSocket_2.54mm:PinSocket_1x03_P2.54mm_Vertical, symbol Connector:Conn_01x03_Pin
- removed J8: FIO1, Connector_PinSocket_2.54mm:PinSocket_1x03_P2.54mm_Vertical, symbol Connector:Conn_01x03_Pin
- removed J9: FIO7, Connector_PinSocket_2.54mm:PinSocket_1x03_P2.54mm_Vertical, symbol Connector:Conn_01x03_Pin
- removed R1, R10, R11, R12, R13, R14, R15, R16, R17, R18, R19, R2, R20, R21, R22, R23, R24, R27, R28, R3, R31, R32, R35, R36, R4, R5, R6, R7, R8, R9: 1k, Resistor_SMD:R_0805_2012Metric_Pad1.20x1.40mm_HandSolder, symbol Device:R_Small
- removed R25, R26, R29, R30, R33, R34: 2k2, Resistor_SMD:R_0805_2012Metric_Pad1.20x1.40mm_HandSolder, symbol Device:R_Small
- removed U1, U2, U3, U4: 74LS04, symbol 74xx:74LS04
- added J30, J31, J32: Conn_01x02_Pin, Connector_PinSocket_2.54mm:PinSocket_1x02_P2.54mm_Vertical, symbol Connector:Conn_01x02_Pin
- added J51, J52, J53, J54, J55, J56: Conn_01x06_Pin, Connector_PinHeader_2.54mm:PinHeader_1x06_P2.54mm_Vertical, symbol Connector:Conn_01x06_Pin
- added J57, J60, J61: Conn_01x04_Pin, Connector_PinHeader_2.54mm:PinHeader_1x04_P2.54mm_Vertical, symbol Connector:Conn_01x04_Pin
- added J58, J59, J62, J63, J64, J65: Conn_01x08_Pin, Connector_PinHeader_2.54mm:PinHeader_1x08_P2.54mm_Vertical, symbol Connector:Conn_01x08_Pin
- J33: value AIN3 -> CIO0
- J34: value AIN6 -> CIO0
- J35: value AIN9 -> CIO0
- R37: value 1k -> 0; now not fitted
Connections:
- net +5V: now also J34.1 (Pin_1), J34.3 (Pin_3), J31.1 (Pin_1), J31.2 (Pin_2), J53.1 (Pin_1), J53.2 (Pin_2), J53.3 (Pin_3), J53.4 (Pin_4), J53.5 (Pin_5), J53.6 (Pin_6), J54.1 (Pin_1), J54.2 (Pin_2), J54.3 (Pin_3), J54.4 (Pin_4), J54.5 (Pin_5), J54.6 (Pin_6), J60.1 (Pin_1), J60.2 (Pin_2), J60.3 (Pin_3), J60.4 (Pin_4), J62.1 (Pin_1), J62.2 (Pin_2), J62.3 (Pin_3), J62.4 (Pin_4), J62.5 (Pin_5), J62.6 (Pin_6), J62.7 (Pin_7), J62.8 (Pin_8), J64.1 (Pin_1), J64.2 (Pin_2), J64.3 (Pin_3), J64.4 (Pin_4), J64.5 (Pin_5), J64.6 (Pin_6), J64.7 (Pin_7), J64.8 (Pin_8); no longer J33.2 (Pin_2)
- net AIN0: now also J51.1 (Pin_1)
- net AIN1: now also J51.2 (Pin_2)
- net AIN10: no longer J47.4 (Pin_4)
- net AIN11: no longer J47.3 (Pin_3)
- net AIN12: no longer J47.2 (Pin_2)
- net AIN13: no longer J47.1 (Pin_1)
- net AIN2: now also J51.3 (Pin_3)
- net AIN3: now also J51.4 (Pin_4); no longer J33.1 (Pin_1)
- net AIN4: now also J51.5 (Pin_5)
- net AIN5: now also J51.6 (Pin_6)
- net AIN6: now also J52.1 (Pin_1); no longer J34.1 (Pin_1)
- net AIN7: now also J52.2 (Pin_2)
- net AIN8: no longer J47.6 (Pin_6)
- net AIN9: no longer J35.2 (Pin_2), J47.5 (Pin_5)
- net CIO0: now also J57.1 (Pin_1)
- net CIO1: now also J57.2 (Pin_2)
- net CIO2: now also J57.3 (Pin_3)
- net CIO3: now also J57.4 (Pin_4)
- net EIO0: now also J58.1 (Pin_1)
- net EIO1: now also J58.2 (Pin_2)
- net EIO2: now also J58.3 (Pin_3)
- net EIO3: now also J58.4 (Pin_4)
- net EIO4: now also J58.5 (Pin_5)
- net EIO5: now also J58.6 (Pin_6)
- net EIO6: now also J58.7 (Pin_7)
- net EIO7: now also J58.8 (Pin_8)
- net FIO0: now also J59.1 (Pin_1)
- net FIO1: now also J59.2 (Pin_2)
- net FIO2: now also J59.3 (Pin_3)
- net FIO3: now also J59.4 (Pin_4)
- net FIO4: now also J59.5 (Pin_5)
- net FIO5: now also J59.6 (Pin_6)
- net FIO6: now also J59.7 (Pin_7)
- net FIO7: now also J59.8 (Pin_8)
- net GND: now also J35.1 (Pin_1), J35.2 (Pin_2), J32.1 (Pin_1), J32.2 (Pin_2), J55.1 (Pin_1), J55.2 (Pin_2), J55.3 (Pin_3), J55.5 (Pin_5), J55.6 (Pin_6), J56.1 (Pin_1), J56.2 (Pin_2), J56.3 (Pin_3), J56.4 (Pin_4), J56.5 (Pin_5), J56.6 (Pin_6), J61.1 (Pin_1), J61.2 (Pin_2), J61.3 (Pin_3), J61.4 (Pin_4), J63.1 (Pin_1), J63.2 (Pin_2), J63.3 (Pin_3), J63.4 (Pin_4), J63.5 (Pin_5), J63.6 (Pin_6), J63.7 (Pin_7), J63.8 (Pin_8), J65.1 (Pin_1), J65.2 (Pin_2), J65.3 (Pin_3), J65.4 (Pin_4), J65.5 (Pin_5), J65.6 (Pin_6), J65.7 (Pin_7), J65.8 (Pin_8); no longer J33.3 (Pin_3), J34.3 (Pin_3)
- net MIO0: now also J33.1 (Pin_1)
- net MIO1: now also J33.2 (Pin_2)
- net MIO2: now also J33.3 (Pin_3)
- new net AIN10_PD: J47.4 (Pin_4), J52.5 (Pin_5)
- new net AIN11_PD: J47.3 (Pin_3), J52.6 (Pin_6)
- new net AIN12_PD: J30.1 (Pin_1), J47.2 (Pin_2)
- new net AIN13_PD: J30.2 (Pin_2), J47.1 (Pin_1)
- new net AIN8_PD: J47.6 (Pin_6), J52.3 (Pin_3)
- new net AIN9_PD: J47.5 (Pin_5), J52.4 (Pin_4)
Other:
- added sheet Analogue Potential Divider (Analogue Potential Divider.kicad_sch)
- added sheet Analogue Potential Divider1 (Analogue Potential Divider.kicad_sch)
- added sheet Analogue Potential Divider2 (Analogue Potential Divider.kicad_sch)
- added sheet Analogue Potential Divider3 (Analogue Potential Divider.kicad_sch)
- added sheet Analogue Potential Divider4 (Analogue Potential Divider.kicad_sch)
- added sheet Analogue Potential Divider5 (Analogue Potential Divider.kicad_sch)
- added sheet LED Indicators (LED Indicators.kicad_sch)
- added sheet LED Indicators1 (LED Indicators.kicad_sch)
- added sheet LED Indicators2 (LED Indicators.kicad_sch)
- added sheet LED Indicators3 (LED Indicators.kicad_sch)
- note added: "need to add caps"
- moved on the sheet: J26, J27, J28, J29, J44, J45, J46, J47, J48, J49, J50, JP1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

Commit message: .
Connections:
- net GND: now also J55.4 (Pin_4)
Other:
- moved on the sheet: J26, J27, J28, J29, J32, J35, J55, J56, J61, J63, J65
